Commit message: Fix 4 wheels Not visible.

File: ros2_ws/src/linorobot2/linorobot2_description/urdf/controllers/ackermann_drive.urdf.xacro (robot description, xacro)
@@ -12,9 +12,7 @@
         <left_steering_joint>front_left_steer_joint</left_steering_joint>
         <right_steering_joint>front_right_steer_joint</right_steering_joint>
-        <!-- 필수 구동 바퀴 조인트 4개 -->
-        <front_left_joint>front_left_wheel_joint</front_left_joint>
-        <front_right_joint>front_right_wheel_joint</front_right_joint>
-        <rear_left_joint>rear_left_wheel_joint</rear_left_joint>
-        <rear_right_joint>rear_right_wheel_joint</rear_right_joint>
+        <!-- 필수 구동 바퀴 조인트 2개 -->
+        <left_joint>rear_left_wheel_joint</left_joint>
+        <right_joint>rear_right_wheel_joint</right_joint>
         <!-- 제원 및 구동 토크 파라미터 -->
         <max_steer>${max_steer_angle}</max_steer>

File: ros2_ws/src/linorobot2/linorobot2_description/urdf/robots/ackermann.urdf.xacro (robot description, xacro)
@@ -9,6 +9,6 @@
   <xacro:property name="wheel_width" value="0.04" />
   <xacro:property name="wheel_pos_x" value="0.18" />  <!-- 휠베이스(전장) 오프셋 -->
-  <xacro:property name="wheel_pos_y" value="0.16" />  <!-- 윤거(트레드) 오프셋 -->
-  <xacro:property name="wheel_pos_z" value="-0.02" />
+  <xacro:property name="wheel_pos_y" value="0.18" />  <!-- 윤거(트레드) 오프셋 -->
+  <xacro:property name="wheel_pos_z" value="-0.05" />
   <xacro:property name="wheel_mass" value="0.5" />
   <xacro:property name="max_steer_angle" value="0.523599" /> <!-- 최대 조향각 약 30도 -->
@@ -74,10 +74,4 @@
         </material>
       </visual>
-      <collision>
-        <origin xyz="0 0 0" rpy="0 0 0"/>
-        <geometry>
-          <box size="0.02 0.02 0.02"/>
-        </geometry>
-      </collision>
       <inertial>
         <origin xyz="0 0 0" rpy="0 0 0"/>
@@ -120,11 +114,5 @@
     </link>
     <gazebo reference="${side}_wheel_link">
-      <visual>
-        <material>
-          <ambient>0.1764 0.4588 0.8509 1.0</ambient>
-          <diffuse>0.1764 0.4588 0.8509 1.0</diffuse>
-          <specular>0.1764 0.4588 0.8509 1.0</specular>
-        </material>
-      </visual>
+      <material>Gazebo/Blue</material>
       <mu1>100.0</mu1>
       <mu2>100.0</mu2>
@@ -154,3 +142,14 @@
     max_steer_angle="${max_steer_angle}"
   />
+  <gazebo>
+    <plugin name="gazebo_ros_joint_state_publisher" filename="libgazebo_ros_joint_state_publisher.so">
+       <update_rate>30</update_rate>
+      <joint_name>front_left_steer_joint</joint_name>
+      <joint_name>front_right_steer_joint</joint_name>
+      <joint_name>front_left_wheel_joint</joint_name>
+      <joint_name>front_right_wheel_joint</joint_name>
+      <joint_name>rear_left_wheel_joint</joint_name>
+      <joint_name>rear_right_wheel_joint</joint_name>
+    </plugin>
+  </gazebo>
 </robot>

Commit message: Fixing do not control the vihicle by keyboard. but not complete.

File: ros2_ws/src/linorobot2/linorobot2_description/urdf/controllers/ackermann_drive.urdf.xacro (robot description, xacro)
@@ -6,13 +6,17 @@
         <ros>
           <remapping>cmd_vel:=/cmd_vel</remapping>
-          <remapping>odom:=/odom</remapping>
+          <!-- <remapping>odom:=/odom</remapping> -->
+          <remapping>odom:=odom/unfiltered</remapping>
         </ros>
         <update_rate>100.0</update_rate>
-        <!-- 필수 조향 조인트 2개 -->
+        <!-- 필수 조향 조인트 2개 및 스티어링 휠 조인트 1개 -->
         <left_steering_joint>front_left_steer_joint</left_steering_joint>
         <right_steering_joint>front_right_steer_joint</right_steering_joint>
-        <!-- 필수 구동 바퀴 조인트 2개 -->
-        <left_joint>rear_left_wheel_joint</left_joint>
-        <right_joint>rear_right_wheel_joint</right_joint>
+        <!-- <steering_wheel_joint>steering_wheel_joint</steering_wheel_joint> -->
+        <!-- 필수 구동/회전 바퀴 조인트 4개 -->
+        <front_left_joint>front_left_wheel_joint</front_left_joint>
+        <front_right_joint>front_right_wheel_joint</front_right_joint>
+        <rear_left_joint>rear_left_wheel_joint</rear_left_joint>
+        <rear_right_joint>rear_right_wheel_joint</rear_right_joint>
         <!-- 제원 및 구동 토크 파라미터 -->
         <max_steer>${max_steer_angle}</max_steer>
@@ -20,19 +24,26 @@
         <max_speed>20.0</max_speed>
         <max_torque>500.0</max_torque>
-        <!-- PID 게인 파라미터 -->
-        <left_steering_pid_gain>1500 0 1</left_steering_pid_gain>
-        <left_steering_i_limit>0 0</left_steering_i_limit>
-        <right_steering_pid_gain>1500 0 1</right_steering_pid_gain>
-        <right_steering_i_limit>0 0</right_steering_i_limit>
-        <linear_velocity_pid_gain>1000 0 1</linear_velocity_pid_gain>
-        <linear_velocity_i_limit>0 0</linear_velocity_i_limit>
+        <!-- PID 게인 파라미터 (소형 차체에 맞춘 적정 물리 게인) -->
+        <left_steering_pid_gain>10 0 0.1</left_steering_pid_gain>
+        <!-- <left_steering_i_limit>0 0</left_steering_i_limit> -->
+        <left_steering_i_range>0 0</left_steering_i_range>
+        <right_steering_pid_gain>10 0 0.1</right_steering_pid_gain>
+        <!-- <right_steering_i_limit>0 0</right_steering_i_limit> -->
+        <right_steering_i_range>0 0</right_steering_i_range>
+        <linear_velocity_pid_gain>10 0 0.1</linear_velocity_pid_gain>
+        <!-- <linear_velocity_i_limit>0 0</linear_velocity_i_limit> -->
+        <linear_velocity_i_range>0 0</linear_velocity_i_range>
         <wheel_separation>${wheel_separation}</wheel_separation>
         <wheel_diameter>${wheel_diameter}</wheel_diameter>
+        <wheel_base>${wheel_base}</wheel_base>
         <!-- 오도메트리 퍼블리시 설정 -->
         <publish_odom>true</publish_odom>
-        <publish_odom_tf>true</publish_odom_tf>
+        <!-- <publish_odom_tf>true</publish_odom_tf> -->
+        <publish_odom_tf>false</publish_odom_tf>
         <publish_wheel_tf>true</publish_wheel_tf>
+        <!-- <publish_wheel_tf>false</publish_wheel_tf> -->
         <odometry_frame>odom</odometry_frame>
         <robot_base_frame>base_footprint</robot_base_frame>
+        <!-- <robot_base_frame>base_link</robot_base_frame> -->
       </plugin>
     </gazebo>

File: ros2_ws/src/linorobot2/linorobot2_description/urdf/robots/ackermann.urdf.xacro (robot description, xacro)
@@ -50,13 +50,13 @@
   <!-- 후륜 구동 바퀴 지면 마찰력(Traction) 설정 -->
   <gazebo reference="rear_left_wheel_link">
-    <mu1>100.0</mu1>
-    <mu2>100.0</mu2>
-    <kp>10000000.0</kp>
+    <mu1>1.0</mu1>
+    <mu2>1.0</mu2>
+    <kp>100000.0</kp>
     <kd>1.0</kd>
   </gazebo>
   <gazebo reference="rear_right_wheel_link">
-    <mu1>100.0</mu1>
-    <mu2>100.0</mu2>
-    <kp>10000000.0</kp>
+    <mu1>1.0</mu1>
+    <mu2>1.0</mu2>
+    <kp>100000.0</kp>
     <kd>1.0</kd>
   </gazebo>
@@ -87,4 +87,5 @@
       <axis xyz="0 0 1"/>
       <limit lower="-${max_steer_angle}" upper="${max_steer_angle}" effort="10.0" velocity="5.0"/>
+      <dynamics damping="0.1" friction="0.1"/>
     </joint>
     <!-- 전륜 바퀴 링크 -->
@@ -115,7 +116,7 @@
     <gazebo reference="${side}_wheel_link">
       <material>Gazebo/Blue</material>
-      <mu1>100.0</mu1>
-      <mu2>100.0</mu2>
-      <kp>10000000.0</kp>
+      <mu1>1.0</mu1>
+      <mu2>1.0</mu2>
+      <kp>100000.0</kp>
       <kd>1.0</kd>
     </gazebo>
@@ -132,4 +133,37 @@
   <xacro:front_steer_wheel side="front_left" pos_x="${wheel_pos_x}" pos_y="${wheel_pos_y}" pos_z="${wheel_pos_z}" />
   <xacro:front_steer_wheel side="front_right" pos_x="${wheel_pos_x}" pos_y="${-wheel_pos_y}" pos_z="${wheel_pos_z}" />
+  <!-- 스티어링 휠 (운전대 핸들) - 차체 상단 대시보드 위치에 형상 추가 -->
+  <!-- <link name="steering_wheel_link">
+    <visual>
+      <origin xyz="0 0 0" rpy="0 0 0"/>
+      <geometry>
+        <cylinder radius="0.06" length="0.01"/>
+      </geometry>
+      <material name="black">
+        <color rgba="0.1 0.1 0.1 1.0"/>
+      </material>
+    </visual>
+    <collision>
+      <origin xyz="0 0 0" rpy="0 0 0"/>
+      <geometry>
+        <cylinder radius="0.06" length="0.01"/>
+      </geometry>
+    </collision>
+    <inertial>
+      <origin xyz="0 0 0" rpy="0 0 0"/>
+      <mass value="0.1"/>
+      <inertia ixx="0.0001" ixy="0" ixz="0" iyy="0.0001" iyz="0" izz="0.0001"/>
+    </inertial>
+  </link>
+  <gazebo reference="steering_wheel_link">
+    <material>Gazebo/Black</material>
+  </gazebo>
+  <joint name="steering_wheel_joint" type="revolute">
+    <parent link="base_link"/>
+    <child link="steering_wheel_link"/>
+    <origin xyz="0.05 0 0.1" rpy="0 -0.5 0"/>
+    <axis xyz="0 0 1"/>
+    <limit lower="-3.14" upper="3.14" effort="10.0" velocity="10.0"/>
+  </joint> -->
   <!-- 4. 센서 및 아커만 플러그인 로드 -->
   <xacro:imu/>
@@ -151,4 +185,5 @@
       <joint_name>rear_left_wheel_joint</joint_name>
       <joint_name>rear_right_wheel_joint</joint_name>
+      <!-- <joint_name>steering_wheel_joint</joint_name> -->
     </plugin>
   </gazebo>
