Commit message: Fix AgileX vehicle model position.

File: ros2_ws/src/hunter_robot/hunter_description/description/hunter_core.urdf.xacro (robot description, xacro)
@@ -20,5 +20,6 @@
     <link name="${prefix}base_link">
       <visual>
-        <origin xyz="-0.05 0 0.12" rpy="0 0 0" />  <!-- HERREEEEE--> <!-- 0.18-->
+        <!-- <origin xyz="-0.05 0 0.12" rpy="0 0 0" />  HERREEEEE 0.18 -->
+        <origin xyz="-0.05 0 0.18" rpy="0 0 0" />
         <geometry>
           <!-- <mesh filename="package://husky_description/meshes/base_link.dae" /> -->

File: ros2_ws/src/hunter_robot/hunter_description/description/wheel.urdf.xacro (robot description, xacro)
@@ -26,5 +26,6 @@
         <origin xyz="0 0 0" rpy="${M_PI/2} 0 0" />
         <geometry>
-          <cylinder length="${wheel_length}" radius="${wheel_radius}" />
+          <!-- <cylinder length="${wheel_length}" radius="${wheel_radius}" /> -->
+          <cylinder length="${wheel_length * 0.6}" radius="${wheel_radius * 0.6}" />
         </geometry>
       </collision>

Commit message: Fixed not working ackermann_drive.

File: ros2_ws/src/hunter_robot/hunter_description/description/hunter_core.urdf.xacro (robot description, xacro)
@@ -44,5 +44,6 @@
     <link name="${prefix}base_footprint"/>
     <joint name="${prefix}base_footprint_joint" type="fixed">
-      <origin xyz="0 0 ${wheel_vertical_offset - wheel_radius}" rpy="0 0 0" />
+      <!-- <origin xyz="0 0 ${wheel_vertical_offset - wheel_radius}" rpy="0 0 0" /> -->
+      <origin xyz="0 0 ${wheel_vertical_offset - wheel_radius * 0.6}" rpy="0 0 0" />
       <parent link="${prefix}base_link" />
       <child link="${prefix}base_footprint" />
@@ -61,6 +62,11 @@
       <child link="${prefix}inertial_link" />
     </joint>
-    <xacro:hunter_wheel wheel_prefix="${prefix}front_left" x="${wheelbase/2}" y="${track/2}" z="${wheel_vertical_offset}" is_sim="${is_sim}"/>
-    <xacro:hunter_wheel wheel_prefix="${prefix}front_right" x="${wheelbase/2}" y="${-track/2}" z="${wheel_vertical_offset}" is_sim="${is_sim}"/>
+    <!-- 기존 코드 -->
+    <!-- <xacro:hunter_wheel wheel_prefix="${prefix}front_left" x="${wheelbase/2}" y="${track/2}" z="${wheel_vertical_offset}" is_sim="${is_sim}"/>
+    <xacro:hunter_wheel wheel_prefix="${prefix}front_right" x="${wheelbase/2}" y="${-track/2}" z="${wheel_vertical_offset}" is_sim="${is_sim}"/> -->
+    <!-- [수정/추가 코드] 전륜 바퀴 2개는 조향 매크로(hunter_steering_wheel) 사용 for Ackermann steering -->
+    <xacro:hunter_steering_wheel wheel_prefix="${prefix}front_left" x="${wheelbase/2}" y="${track/2}" z="${wheel_vertical_offset}" is_sim="${is_sim}"/>
+    <xacro:hunter_steering_wheel wheel_prefix="${prefix}front_right" x="${wheelbase/2}" y="${-track/2}" z="${wheel_vertical_offset}" is_sim="${is_sim}"/>
+    <!-- 후륜 바퀴 (속도 제어) -->
     <xacro:hunter_wheel wheel_prefix="${prefix}back_left" x="${-wheelbase/2}" y="${track/2}" z="${wheel_vertical_offset}" is_sim="${is_sim}"/>
     <xacro:hunter_wheel wheel_prefix="${prefix}back_right" x="${-wheelbase/2}" y="${-track/2}" z="${wheel_vertical_offset}" is_sim="${is_sim}"/>

File: ros2_ws/src/hunter_robot/hunter_description/description/ros2_control.xacro (robot description, xacro)
@@ -5,5 +5,6 @@
             <plugin>gazebo_ros2_control/GazeboSystem</plugin>
         </hardware>
-        <joint name="front_right_wheel_joint">
+        <!-- [기존코드] 후륜 구동 바퀴 (속도 제어: velocity) -->
+        <!-- <joint name="front_right_wheel_joint">
             <command_interface name="velocity">
                 <param name="min">-10</param>
@@ -20,5 +21,15 @@
             <state_interface name="velocity"/>
             <state_interface name="position"/>
+        </joint> -->
+        <!-- [추가 코드 for 아크만 조향] 전륜 조향 관절 (각도 제어: position 추가) 🌟 -->
+        <joint name="front_left_steering_joint">
+            <command_interface name="position"/>
+            <state_interface name="position"/>
         </joint>
+        <joint name="front_right_steering_joint">
+            <command_interface name="position"/>
+            <state_interface name="position"/>
+        </joint>
+        <!-- 후륜 구동 바퀴 (속도 제어: velocity) -->
         <joint name="back_right_wheel_joint">
             <command_interface name="velocity">
@@ -48,4 +59,5 @@
             <!-- 🌟 새로 만든 ackermann_controllers.yaml 파일로 경로 지정 -->
             <parameters>$(find hunter_gazebo)/config/ackermann_controllers.yaml</parameters>
+            <!-- 🌟 /cmd_vel 토픽을 아커만 컨트롤러로 자동 연결하는 리매핑 추가 -->
             <ros>
                 <remapping>/ackermann_steering_controller/reference_unstamped:=/cmd_vel</remapping>

File: ros2_ws/src/hunter_robot/hunter_description/description/wheel.urdf.xacro (robot description, xacro)
@@ -26,5 +26,6 @@
         <origin xyz="0 0 0" rpy="${M_PI/2} 0 0" />
         <geometry>
-          <!-- <cylinder length="${wheel_length}" radius="${wheel_radius}" /> -->
+          <!-- [기존 코드] <cylinder length="${wheel_length}" radius="${wheel_radius}" /> -->
+          <!-- [수정 코드] 메쉬 크기(0.6)에 맞춰 충돌체 크기 비율 조정 -->
           <cylinder length="${wheel_length * 0.6}" radius="${wheel_radius * 0.6}" />
         </geometry>
@@ -43,5 +44,5 @@
       <kp value="10000000.0" />
       <kd value="1.0" />
-      <fdir1 value="1 0 0"/>
+      <!-- <fdir1 value="1 0 0"/> -->
     </gazebo>
   </xacro:if>
@@ -55,3 +56,57 @@
   </xacro:unless>
   </xacro:macro>
+    <!-- [새로 추가: 전륜 조향 바퀴 매크로 - Z축 조향 관절 + Y축 구동 관절] 🌟 -->
+  <xacro:macro name="hunter_steering_wheel" params="wheel_prefix x y z roll:=0.0 pitch:=0.0 yaw:=0.0 is_sim:=true">
+    <!-- 조향 킹핀 링크 (Dummy Steering Link) -->
+    <link name="${wheel_prefix}_steering_link">
+      <inertial>
+        <mass value="0.5" />
+        <origin xyz="0 0 0" />
+        <inertia ixx="0.001" ixy="0" ixz="0" iyy="0.001" iyz="0" izz="0.001" />
+      </inertial>
+    </link>
+    <!-- 1. Z축 조향 관절 (base_link -> steering_link) -->
+    <joint name="${wheel_prefix}_steering_joint" type="revolute">
+      <parent link="base_link"/>
+      <child link="${wheel_prefix}_steering_link"/>
+      <origin xyz="${x} ${y} ${z}" rpy="${roll} ${pitch} ${yaw}"/>
+      <axis xyz="0 0 1"/>
+      <limit lower="-1.2" upper="1.2" effort="100.0" velocity="2.0"/>
+      <dynamics damping="1.0" friction="0.1"/>
+    </joint>
+    <!-- 바퀴 링크 -->
+    <link name="${wheel_prefix}_wheel">
+      <inertial>
+        <mass value="2.637" />
+        <origin xyz="0 0 0" />
+        <inertia ixx="0.02467" ixy="0" ixz="0" iyy="0.04411" iyz="0" izz="0.02467" />
+      </inertial>
+      <visual>
+        <origin xyz="0 0 0" rpy="0 0 0" />
+        <geometry>
+          <mesh filename="file://$(find hunter_description)/meshes/wheel.dae" scale="0.6 0.6 0.6"/>
+        </geometry>
+      </visual>
+      <collision>
+        <origin xyz="0 0 0" rpy="${M_PI/2} 0 0" />
+        <geometry>
+          <cylinder length="${wheel_length * 0.6}" radius="${wheel_radius * 0.6}" />
+        </geometry>
+      </collision>
+    </link>
+    <!-- 2. Y축 바퀴 회전 관절 (steering_link -> wheel) -->
+    <joint name="${wheel_prefix}_wheel_joint" type="continuous">
+      <parent link="${wheel_prefix}_steering_link"/>
+      <child link="${wheel_prefix}_wheel"/>
+      <origin xyz="0 0 0" rpy="0 0 0"/>
+      <axis xyz="0 1 0"/>
+    </joint>
+    <gazebo reference="${wheel_prefix}_wheel">
+      <mu1 value="0.5"/>
+      <mu2 value="0.5"/>
+      <kp value="10000000.0" />
+      <kd value="1.0" />
+      <!-- <fdir1 value="1 0 0"/> -->
+    </gazebo>
+  </xacro:macro>
 </robot>
