Commit message: Fixed slam_rotation issue.

File: ros2_ws/src/hunter_robot/hunter_description/description/hunter.urdf.xacro (robot description, xacro)
@@ -12,5 +12,5 @@
     </xacro:if>
     <xacro:unless value="$(arg use_ros2_control)">
-        <xacro:include filename="$(find hunter_description)/description/gazebo_control.xacro" />
+        <!-- <xacro:include filename="$(find hunter_description)/description/gazebo_control.xacro" /> -->
     </xacro:unless>
 </robot>

File: ros2_ws/src/hunter_robot/hunter_description/description/ros2_control.xacro (robot description, xacro)
@@ -6,20 +6,21 @@
         </hardware>
         <!-- [기존코드] 후륜 구동 바퀴 (속도 제어: velocity) -->
-        <!-- <joint name="front_right_wheel_joint">
-            <command_interface name="velocity">
+        <!-- 전륜 바퀴 (조향에 의해 굴러가는 passive joint) -->
+        <joint name="front_right_wheel_joint">
+            <!-- <command_interface name="velocity">
                 <param name="min">-10</param>
                 <param name="max">10</param>
-            </command_interface>
+            </command_interface> -->
             <state_interface name="velocity"/>
             <state_interface name="position"/>
         </joint>
         <joint name="front_left_wheel_joint">
-            <command_interface name="velocity">
+            <!-- <command_interface name="velocity">
                 <param name="min">-10</param>
                 <param name="max">10</param>
-            </command_interface>
+            </command_interface> -->
             <state_interface name="velocity"/>
             <state_interface name="position"/>
-        </joint> -->
+        </joint>
         <!-- [추가 코드 for 아크만 조향] 전륜 조향 관절 (각도 제어: position 추가) 🌟 -->
         <joint name="front_left_steering_joint">

File: ros2_ws/src/hunter_robot/hunter_description/description/wheel.urdf.xacro (robot description, xacro)
@@ -38,8 +38,9 @@
       <origin xyz="${x} ${y} ${z}" rpy="${roll} ${pitch} ${yaw}"/>
       <axis xyz="0 1 0" rpy="0 0 0" />
+      <limit effort="100.0" velocity="20.0"/>
     </joint>
     <gazebo reference="${wheel_prefix}_wheel">
-      <mu1 value="10.0"/>   <!-- 0.5 -> 10.0 상향 -->
-      <mu2 value="10.0"/>   <!-- 0.5 -> 10.0 상향 -->
+      <mu1 value="100.0"/>   <!-- 0.5 -> 100.0 상향 -->
+      <mu2 value="100.0"/>   <!-- 0.5 -> 100.0 상향 -->
       <kp value="10000000.0" />
       <kd value="1.0" />
@@ -101,8 +102,9 @@
       <origin xyz="0 0 0" rpy="0 0 0"/>
       <axis xyz="0 1 0"/>
+      <limit effort="100.0" velocity="20.0"/>
     </joint>
     <gazebo reference="${wheel_prefix}_wheel">
-      <mu1 value="10.0"/>   <!-- 0.5 -> 10.0 상향 🌟 -->
-      <mu2 value="10.0"/>   <!-- 0.5 -> 10.0 상향 🌟 -->
+      <mu1 value="100.0"/>   <!-- 10.0 -> 100.0 상향 (슬립 방지) 🌟 -->
+      <mu2 value="100.0"/>   <!-- 10.0 -> 100.0 상향 (슬립 방지) 🌟 -->
       <kp value="10000000.0" />
       <kd value="1.0" />
